Commit message: Cartographer without IMU

File: cartographer_configs/radmap.urdf (robot description, URDF)
Before this commit: robot cartographer_backpack_3d, 4 links, 3 joints
Links:
- removed link horizontal_vlp16_link
- removed link imu_link
- removed link vertical_vlp16_link
- added link novatel; visual box size=0.0 0.0 0.0
- added link velodyne_port; visual cylinder length=0.0 radius=0.0
- added link velodyne_starboard; visual cylinder length=0.0 radius=0.0
Joints:
- removed joint horizontal_vlp16_link_joint
- removed joint imu_link_joint
- removed joint vertical_vlp16_link_joint
- added joint novatel_joint: type fixed, parent base_link, child novatel, origin xyz=0 0 0 rpy=0 0 0
- added joint velodyne_port_joint: type fixed, parent base_link, child velodyne_port, origin xyz=-1.224 0.376 -0.070 rpy=0.031 0.197 1.506
- added joint velodyne_starboard_joint: type fixed, parent base_link, child velodyne_starboard, origin xyz=1.350 0.200 -0.120 rpy=-0.018 -0.197 -1.569
